Commit message: [camera] feat: 添加更多吊射相关参数，完善吊射切换相机源功能，添加吊射相机的 urdf 描述。

File: src/rm_gimbal_description/urdf/rm_gimbal.urdf.xacro (robot description, xacro)
@@ -4,4 +4,6 @@
   <xacro:arg name="xyz" default="0.10 0 0.05" />
   <xacro:arg name="rpy" default="0 0 0" />
+  <xacro:arg name="lob_xyz" default="0 0 0" />
+  <xacro:arg name="lob_rpy" default="0 0 0" />
   <link name="gimbal_odom" />
   <link name="yaw_link" />
@@ -30,3 +32,16 @@
     <child link="camera_optical_frame" />
   </joint>
+  <!-- new two-layer lob camera frame -->
+  <link name="camera_lob_link" />
+  <joint name="camera_lob_joint" type="fixed">
+    <origin xyz="$(arg lob_xyz)" rpy="$(arg lob_rpy)" />
+    <parent link="yaw_link" />
+    <child link="camera_lob_link" />
+  </joint>
+  <link name="camera_optical_frame_lob" />
+  <joint name="camera_optical_joint_lob" type="fixed">
+    <origin xyz="0 0 0" rpy="${-pi/2} 0 ${-pi/2}" />
+    <parent link="camera_lob_link" />
+    <child link="camera_optical_frame_lob" />
+  </joint>
 </robot>

Commit message: feat: 添加相机标定脚本，优化相机启动逻辑，更新目标消息格式，修正云台 URDF 文件

File: src/rm_gimbal_description/urdf/rm_gimbal.urdf.xacro (robot description, xacro)
@@ -17,5 +17,5 @@
     <parent link="yaw_link" />
     <child link="pitch_link" />
-    <axis xyz="0 -1 0" />
+    <axis xyz="0 1 0" />
   </joint>
   <link name="camera_link" />

Commit message: 拍视频用的稳定版

File: src/rm_gimbal_description/urdf/rm_gimbal.urdf.xacro (robot description, xacro)
@@ -15,5 +15,5 @@
     <parent link="yaw_link" />
     <child link="pitch_link" />
-    <axis xyz="0 -1 0" />
+    <axis xyz="0 1 0" />
   </joint>
   <link name="camera_link" />
